Commit message: Initial

File: src/modelling/urdf/follower/follower.urdf (robot description, URDF)
Before this commit: robot follower, 7 links, 6 joints
Links:
- link base_link: geometry collision mesh filename=package://src/modelling/urdf/follower/meshes/base_link.STL; collision mesh filename=package://src/modelling/urdf/follower/meshes/base_link_moto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
- link link_1: geometry collision mesh filename=package://src/modelling/urdf/follower/meshes/link_1.STL; collision mesh filename=package://src/modelling/urdf/follower/meshes/link_1_motor.S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
- link link_2: geometry collision mesh filename=package://src/modelling/urdf/follower/meshes/link_2.STL; collision mesh filename=package://src/modelling/urdf/follower/meshes/link_2_motor.S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
- link link_3: geometry collision mesh filename=package://src/modelling/urdf/follower/meshes/link_3.STL; collision mesh filename=package://src/modelling/urdf/follower/meshes/link_3_motor.S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
- link link_4: geometry collision mesh filename=package://src/modelling/urdf/follower/meshes/link_4.STL; collision mesh filename=package://src/modelling/urdf/follower/meshes/link_4_motor.S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
- link link_5: geometry collision mesh filename=package://src/modelling/urdf/follower/meshes/link_5.STL; collision mesh filename=package://src/modelling/urdf/follower/meshes/link_5_motor.S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
- link link_6: geometry collision mesh filename=package://src/modelling/urdf/follower/meshes/link_6.STL; visual mesh filename=package://src/modelling/urdf/follower/meshes/link_6.STL
