Commit message: Initial

File: src/simulation/urdf/ball/redball.urdf (robot description, URDF)
Before this commit: robot myfirst, 1 links, 0 joints
Links:
- link base_link: geometry visual sphere radius=0.3

Commit message: Initial

File: src/simulation/urdf/ball/redball.urdf (robot description, URDF)
Before this commit: robot myfirst, 1 links, 0 joints
Links:
- link base_link: geometry visual sphere radius=0.1

Commit message: Initial

File: src/simulation/urdf/ball/redball.urdf (robot description, URDF)
Before this commit: robot myfirst, 1 links, 0 joints
Links:
- link base_link: geometry visual sphere radius=0.01

Commit message: Initial

File: src/simulation/urdf/ball/redball.urdf (robot description, URDF)
Before this commit: robot myfirst, 1 links, 0 joints
Links:
- added link world
Joints:
- added joint floating_joint: type floating, parent world, child base_link
